Commit message: working on soft ball env read state

File: assets/objects/hydraulic_press/press.urdf (robot description, URDF)
Before this commit: robot hydraulic_press, 2 links, 1 joints
Links:
- removed link base_link
- removed link child_link
- added link base, mass 2.7; collision box size=0.5 0.5 0.03; visual box size=0.5 0.5 0.03
- added link body, mass 0.2; collision box size=0.5 0.5 0.1; visual box size=0.5 0.5 0.1
- added link world
Joints:
- removed joint press_joint
- added joint body_to_base: type prismatic, parent body, child base, origin xyz=0 0 0.0, axis 0.0 0.0 -1.0, limit lower=-0.2 upper=0.2 effort=1000.0 velocity=1
- added joint world_to_body: type fixed, parent world, child body, origin xyz=0 0 0.0
