Commit message: working clasical pick and place algorithm using neural network

File: assets/objects/UR5/urdf/ur5_robotiq_140_modified.urdf (robot description, URDF)
Before this commit: robot ur5_robotiq_140, 20 links, 19 joints
Joints:
- joint wrist_3_joint: limit lower=-3.14159265359 upper=3.14159265359 effort=28.0 velocity=3.2 -> lower=-31.4159265359 upper=31.4159265359 effort=28.0 velocity=3.2
