Commit message: resize boxes

File: assets/objects/box/urdf/box_dark.urdf (robot description, URDF)
Before this commit: robot box_dark, 5 links, 4 joints
Links:
- link box_bottom: geometry collision box size=0.3 0.3 0.02; visual box size=0.3 0.3 0.02
- link box_wall_back: geometry collision box size=0.3 0.02 0.25; visual box size=0.3 0.02 0.25
- link box_wall_front: geometry collision box size=0.3 0.02 0.25; visual box size=0.3 0.02 0.25
- link box_wall_left: geometry collision box size=0.02 0.34 0.25; visual box size=0.02 0.34 0.25
- link box_wall_right: geometry collision box size=0.02 0.34 0.25; visual box size=0.02 0.34 0.25

File: assets/objects/box/urdf/box_dark_gray.urdf (robot description, URDF)
Before this commit: robot box_dark, 5 links, 4 joints
Links:
- link box_bottom: geometry collision box size=0.3 0.3 0.02; visual box size=0.3 0.3 0.02
- link box_wall_back: geometry collision box size=0.3 0.02 0.25; visual box size=0.3 0.02 0.25
- link box_wall_front: geometry collision box size=0.3 0.02 0.25; visual box size=0.3 0.02 0.25
- link box_wall_left: geometry collision box size=0.02 0.34 0.25; visual box size=0.02 0.34 0.25
- link box_wall_right: geometry collision box size=0.02 0.34 0.25; visual box size=0.02 0.34 0.25

File: assets/objects/box/urdf/box_light.urdf (robot description, URDF)
Before this commit: robot box_light, 5 links, 4 joints
Links:
- link box_bottom: geometry collision box size=0.3 0.3 0.02; visual box size=0.3 0.3 0.02
- link box_wall_back: geometry collision box size=0.3 0.02 0.25; visual box size=0.3 0.02 0.25
- link box_wall_front: geometry collision box size=0.3 0.02 0.25; visual box size=0.3 0.02 0.25
- link box_wall_left: geometry collision box size=0.02 0.34 0.25; visual box size=0.02 0.34 0.25
- link box_wall_right: geometry collision box size=0.02 0.34 0.25; visual box size=0.02 0.34 0.25

File: assets/objects/box/urdf/box_light_gray.urdf (robot description, URDF)
Before this commit: robot box_light, 5 links, 4 joints
Links:
- link box_bottom: geometry collision box size=0.3 0.3 0.02; visual box size=0.3 0.3 0.02
- link box_wall_back: geometry collision box size=0.3 0.02 0.25; visual box size=0.3 0.02 0.25
- link box_wall_front: geometry collision box size=0.3 0.02 0.25; visual box size=0.3 0.02 0.25
- link box_wall_left: geometry collision box size=0.02 0.34 0.25; visual box size=0.02 0.34 0.25
- link box_wall_right: geometry collision box size=0.02 0.34 0.25; visual box size=0.02 0.34 0.25
